File: ClusterBlaster.kicad_pcb (KiCad board)
At the start: 2 copper layers, 65.4 x 50.2 mm, 20 parts, among them J1 OBD2, J2 Cluster Display, SW1 UP, SW2 DOWN, SW3 ENTER, U1 LM339, U2 L7805, U3 Arduino

Commit message: PCB improvements
Routing:
- net K-Line: track 34.6 -> 34.0 mm
Changed lines of the file:
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@@
     (pad_to_mask_clearance 0)
     (pcbplotparams
-      (layerselection 0x0001030_ffffffff)
+      (layerselection 0x00010f0_ffffffff)
       (plot_on_all_layers_selection 0x0000000_00000000)
       (disableapertmacros false)
@@
     (property "ki_keywords" "R res resistor")
     (attr smd)
-    (fp_text reference "R3" (at 3.175 0 90) (layer "F.SilkS")
+    (fp_text reference "R3" (at -3.175 0 90) (layer "F.SilkS")
         (effects (font (size 1 1) (thickness 0.15)))
     )
@@
     (property "ki_keywords" "R res resistor")
     (attr smd)
-    (fp_text reference "R6" (at 2.8975 0) (layer "F.SilkS")
+    (fp_text reference "R6" (at -2.8175 0) (layer "F.SilkS")
         (effects (font (size 1 1) (thickness 0.15)))
     )
@@
     )
   )
+  (gr_line (start 124.968 85.09) (end 119.888 85.09)
+    (stroke (width 0.15) (type default)) (layer "F.SilkS"))
+  (gr_line (start 124.968 83.82) (end 119.888 83.82)
+    (stroke (width 0.15) (type default)) (layer "F.SilkS"))
+  (gr_line (start 124.968 81.28) (end 119.888 81.28)
+    (stroke (width 0.15) (type default)) (layer "F.SilkS"))
+  (gr_line (start 124.968 80.01) (end 119.888 80.01)
+    (stroke (width 0.15) (type default)) (layer "F.SilkS"))
+  (gr_line (start 124.968 82.55) (end 119.888 82.55)
+    (stroke (width 0.15) (type default)) (layer "F.SilkS"))
+  (gr_line (start 124.968 78.74) (end 119.888 78.74)
+    (stroke (width 0.15) (type default)) (layer "F.SilkS"))
   (gr_line (start 128.534583 48.842084) (end 128.556545 48.842046)
     (stroke (width 0.092604) (type solid)) (layer "F.Mask"))
@@
     (effects (font (size 1 1) (thickness 0.25) bold) (justify left bottom))
   )
-  (segment (start 161.29 71.755) (end 161.29 69.98) (width 0.25) (layer "F.Cu") (net 1))
   (segment (start 142.5175 70.1275) (end 138.43 66.04) (width 0.25) (layer "F.Cu") (net 1))
   (segment (start 154.305 70.1275) (end 142.5175 70.1275) (width 0.25) (layer "F.Cu") (net 1))
-  (segment (start 157.48 71.755) (end 158.75 73.025) (width 0.25) (layer "F.Cu") (net 1))
+  (segment (start 158.242 72.39) (end 160.655 72.39) (width 0.25) (layer "F.Cu") (net 1))
+  (segment (start 157.48 71.628) (end 158.242 72.39) (width 0.25) (layer "F.Cu") (net 1))
   (segment (start 157.3325 70.1275) (end 157.48 69.98) (width 0.25) (layer "F.Cu") (net 1))
+  (segment (start 161.29 71.755) (end 161.29 69.98) (width 0.25) (layer "F.Cu") (net 1))
   (segment (start 154.305 70.1275) (end 157.3325 70.1275) (width 0.25) (layer "F.Cu") (net 1))
-  (segment (start 157.48 69.98) (end 157.48 71.755) (width 0.25) (layer "F.Cu") (net 1))
-  (segment (start 158.75 73.025) (end 160.02 73.025) (width 0.25) (layer "F.Cu") (net 1))
-  (segment (start 160.02 73.025) (end 161.29 71.755) (width 0.25) (layer "F.Cu") (net 1))
+  (segment (start 157.48 69.98) (end 157.48 71.628) (width 0.25) (layer "F.Cu") (net 1))
+  (segment (start 160.655 72.39) (end 161.29 71.755) (width 0.25) (layer "F.Cu") (net 1))
   (segment (start 138.43 66.04) (end 138.43 60.626) (width 0.25) (layer "F.Cu") (net 1))
   (segment (start 148.59 62.23) (end 147.32 60.96) (width 0.55) (layer "F.Cu") (net 2))
@@
   (segment (start 147.32 57.51) (end 147.325 57.505) (width 0.55) (layer "F.Cu") (net 2))
   (segment (start 154.94 62.23) (end 148.59 62.23) (width 0.55) (layer "F.Cu") (net 2))
+  (segment (start 160.02 68.58) (end 155.751117 64.311117) (width 0.55) (layer "F.Cu") (net 2))
   (segment (start 147.32 60.96) (end 147.32 57.51) (width 0.55) (layer "F.Cu") (net 2))
-  (segment (start 160.02 69.98) (end 160.02 69.391117) (width 0.55) (layer "F.Cu") (net 2))
   (segment (start 154.94 80.01) (end 157.56 80.01) (width 0.55) (layer "F.Cu") (net 2))
   (segment (start 160.02 69.98) (end 160.02 69.215) (width 0.55) (layer "F.Cu") (net 2))
   (segment (start 146.73 58.1) (end 147.325 57.505) (width 0.55) (layer "F.Cu") (net 2))
+  (segment (start 160.02 69.98) (end 160.02 68.58) (width 0.55) (layer "F.Cu") (net 2))
   (segment (start 154.94 68.3025) (end 154.94 64.311117) (width 0.55) (layer "F.Cu") (net 2))
-  (segment (start 160.02 69.391117) (end 154.94 64.311117) (width 0.55) (layer "F.Cu") (net 2))
   (segment (start 154.94 64.311117) (end 154.94 62.23) (width 0.55) (layer "F.Cu") (net 2))
   (segment (start 138.43 58.126) (end 144.754 58.126) (width 0.55) (layer "F.Cu") (net 2))
+  (segment (start 155.751117 64.311117) (end 154.94 64.311117) (width 0.55) (layer "F.Cu") (net 2))
   (segment (start 144.78 58.1) (end 146.73 58.1) (width 0.55) (layer "F.Cu") (net 2))
   (segment (start 144.754 58.126) (end 144.78 58.1) (width 0.55) (layer "F.Cu") (net 2))
@@
   (segment (start 159.987437 62.23) (end 164.705 66.947563) (width 0.55) (layer "B.Cu") (net 2))
   (segment (start 164.705 72.15) (end 156.845 80.01) (width 0.55) (layer "B.Cu") (net 2))
-  (via (at 161.29 78.105) (size 0.8) (drill 0.4) (layers "F.Cu" "B.Cu") (free) (net 3))
+  (via (at 160.655 78.105) (size 0.8) (drill 0.4) (layers "F.Cu" "B.Cu") (free) (net 3))
   (via (at 158.75 60.325) (size 0.8) (drill 0.4) (layers "F.Cu" "B.Cu") (free) (net 3))
-  (via (at 175.26 60.96) (size 0.8) (drill 0.4) (layers "F.Cu" "B.Cu") (free) (net 3))
+  (via (at 174.625 62.23) (size 0.8) (drill 0.4) (layers "F.Cu" "B.Cu") (free) (net 3))
   (via (at 168.91 59.055) (size 0.8) (drill 0.4) (layers "F.Cu" "B.Cu") (free) (net 3))
-  (via (at 156.845 64.135) (size 0.8) (drill 0.4) (layers "F.Cu" "B.Cu") (free) (net 3))
-  (via (at 172.085 78.105) (size 0.8) (drill 0.4) (layers "F.Cu" "B.Cu") (free) (net 3))
+  (via (at 157.48 64.135) (size 0.8) (drill 0.4) (layers "F.Cu" "B.Cu") (free) (net 3))
+  (via (at 174.625 78.74) (size 0.8) (drill 0.4) (layers "F.Cu" "B.Cu") (free) (net 3))
   (via (at 149.225 60.325) (size 0.8) (drill 0.4) (layers "F.Cu" "B.Cu") (free) (net 3))
   (segment (start 177.8 56.57) (end 180.34 59.11) (width 0.55) (layer "F.Cu") (net 4))
@@
   (segment (start 157.56 82.55) (end 135.89 82.55) (width 0.25) (layer "F.Cu") (net 5))
   (segment (start 133.94 84.5) (end 133.94 87.845) (width 0.25) (layer "F.Cu") (net 5))
-  (segment (start 158.75 69.98) (end 158.75 71.755) (width 0.25) (layer "F.Cu") (net 5))
   (segment (start 135.89 82.55) (end 133.94 84.5) (width 0.25) (layer "F.Cu") (net 5))
   (segment (start 133.94 90.76) (end 133.985 90.805) (width 0.25) (layer "F.Cu") (net 5))
-  (via (at 158.75 71.755) (size 0.8) (drill 0.4) (layers "F.Cu" "B.Cu") (free) (net 5))
+  (segment (start 158.75 69.98) (end 158.75 71.628) (width 0.25) (layer "F.Cu") (net 5))
+  (via (at 158.75 71.628) (size 0.8) (drill 0.4) (layers "F.Cu" "B.Cu") (free) (net 5))
   (via (at 158.75 76.835) (size 0.8) (drill 0.4) (layers "F.Cu" "B.Cu") (free) (net 5))
   (via (at 133.985 90.805) (size 0.8) (drill 0.4) (layers "F.Cu" "B.Cu") (free) (net 5))
-  (segment (start 158.75 76.835) (end 158.75 71.755) (width 0.25) (layer "B.Cu") (net 5))
   (segment (start 142.24 79.375) (end 144.78 76.835) (width 0.25) (layer "B.Cu") (net 5))
+  (segment (start 158.75 76.835) (end 158.75 71.628) (width 0.25) (layer "B.Cu") (net 5))
   (segment (start 140.209695 90.805) (end 142.24 88.774695) (width 0.25) (layer "B.Cu") (net 5))
   (segment (start 144.78 76.835) (end 158.75 76.835) (width 0.25) (layer "B.Cu") (net 5))
   (segment (start 142.24 88.774695) (end 142.24 79.375) (width 0.25) (layer "B.Cu") (net 5))
   (segment (start 133.985 90.805) (end 140.209695 90.805) (width 0.25) (layer "B.Cu") (net 5))
-  (segment (start 162.56 78.74) (end 161.29 80.01) (width 0.25) (layer "F.Cu") (net 6))
-  (segment (start 161.29 80.01) (end 159.385 80.01) (width 0.25) (layer "F.Cu") (net 6))
+  (segment (start 162.56 78.232) (end 160.782 80.01) (width 0.25) (layer "F.Cu") (net 6))
+  (segment (start 160.782 80.01) (end 159.385 80.01) (width 0.25) (layer "F.Cu") (net 6))
+  (segment (start 162.56 74.93) (end 162.56 78.232) (width 0.25) (layer "F.Cu") (net 6))
   (segment (start 157.48 76.590305) (end 159.385 78.495305) (width 0.25) (layer "F.Cu") (net 6))
-  (segment (start 162.56 74.93) (end 162.56 78.74) (width 0.25) (layer "F.Cu") (net 6))
   (segment (start 157.48 74.93) (end 157.48 76.590305) (width 0.25) (layer "F.Cu") (net 6))
   (segment (start 159.385 78.495305) (end 159.385 80.01) (width 0.25) (layer "F.Cu") (net 6))
